Commit message: Add Mujoco compatibility for RL training with objects

File: src/holosoma/holosoma/data/motions/g1_29dof/whole_body_tracking/objects_largebox.urdf (robot description, URDF)
Before this commit: robot largebox.urdf, 1 links, 0 joints
Links:
- removed link baseLink
- added link link, mass 0.1; collision mesh filename=largebox.obj scale=1.0 1.0 1.0; visual mesh filename=largebox.obj scale=1.0 1.0 1.0
