Commit message: tune(wbt): increase largebox mass 0.1 -> 0.811 for sim2sim realism

File: src/holosoma/holosoma/data/motions/g1_29dof/whole_body_tracking/objects_largebox.urdf (robot description, URDF)
Before this commit: robot largebox.urdf, 1 links, 0 joints
Links:
- link baseLink: mass 0.1 -> 0.811
