Commit message: fix(g1): align training URDF ankle limits to native unitree_description (effort 50->35, vel 37->30)
The 4 ankle joints (pitch/roll, left/right) in the G1 27/29-DOF training URDFs used
effort=50/velocity=37, while the native unitree_description g1.urdf uses effort=35/velocity=30.
Align training to the deployment robot's native limits so the policy is trained within the
actuators' real bounds. Position limits, axes and all other joints unchanged.

File: src/holosoma/holosoma/data/robots/g1/g1_27dof.urdf (robot description, URDF)
Before this commit: robot g1, 42 links, 41 joints
Joints:
- joint left_ankle_pitch_joint: limit lower=-0.87267 upper=0.5236 effort=50 velocity=37 -> lower=-0.87267 upper=0.5236 effort=35 velocity=30
- joint left_ankle_roll_joint: limit lower=-0.2618 upper=0.2618 effort=50 velocity=37 -> lower=-0.2618 upper=0.2618 effort=35 velocity=30
- joint right_ankle_pitch_joint: limit lower=-0.87267 upper=0.5236 effort=50 velocity=37 -> lower=-0.87267 upper=0.5236 effort=35 velocity=30
- joint right_ankle_roll_joint: limit lower=-0.2618 upper=0.2618 effort=50 velocity=37 -> lower=-0.2618 upper=0.2618 effort=35 velocity=30

File: src/holosoma/holosoma/data/robots/g1/g1_29dof.urdf (robot description, URDF)
Before this commit: robot g1, 42 links, 41 joints
Joints:
- joint left_ankle_pitch_joint: limit lower=-0.87267 upper=0.5236 effort=50 velocity=37 -> lower=-0.87267 upper=0.5236 effort=35 velocity=30
- joint left_ankle_roll_joint: limit lower=-0.2618 upper=0.2618 effort=50 velocity=37 -> lower=-0.2618 upper=0.2618 effort=35 velocity=30
- joint right_ankle_pitch_joint: limit lower=-0.87267 upper=0.5236 effort=50 velocity=37 -> lower=-0.87267 upper=0.5236 effort=35 velocity=30
- joint right_ankle_roll_joint: limit lower=-0.2618 upper=0.2618 effort=50 velocity=37 -> lower=-0.2618 upper=0.2618 effort=35 velocity=30

Commit message: feat(g1): add battery + d435 payload links to training URDF to match real robot
Port the battery (2.5 kg, fixed to imu_in_torso) and d435 camera frame (massless, fixed
to torso_link) from the native unitree_description g1.urdf into the G1 27/29-DOF training
URDFs. The training model was 2.5 kg lighter than the real robot and missing the battery's
torso mass/inertia; aligning it reduces the sim-to-real mass/CoM gap. Total link mass now
35.84 kg, matching the deployment model.

File: src/holosoma/holosoma/data/robots/g1/g1_27dof.urdf (robot description, URDF)
Before this commit: robot g1, 42 links, 41 joints
Links:
- added link battery, mass 2.5
- added link d435_link
Joints:
- added joint battery_joint: type fixed, parent imu_in_torso, child battery, origin xyz=0.05 0.025 -0.01 rpy=0 0 0
- added joint d435_joint: type fixed, parent torso_link, child d435_link, origin xyz=0.0576235 0.01753 0.42987 rpy=0 0.8307767239493009 0

File: src/holosoma/holosoma/data/robots/g1/g1_29dof.urdf (robot description, URDF)
Before this commit: robot g1, 42 links, 41 joints
Links:
- added link battery, mass 2.5
- added link d435_link
Joints:
- added joint battery_joint: type fixed, parent imu_in_torso, child battery, origin xyz=0.05 0.025 -0.01 rpy=0 0 0
- added joint d435_joint: type fixed, parent torso_link, child d435_link, origin xyz=0.0576235 0.01753 0.42987 rpy=0 0.8307767239493009 0
