Commit message: fix(g1): align remaining G1 URDFs to real robot (ankle limits; battery+d435 on sim asset)
Apply the same real-robot alignment to the rest of the G1 URDFs:
- main_mesh_collision_halfspherehand.urdf (a sim robot asset referenced in robot configs):
  ankle limits 50/37 -> 35/30, plus battery (2.5 kg, imu_in_torso) and d435 camera frame.
- retargeting models g1_27dof/g1_29dof/g1_29dof_spherehand.urdf: ankle limits 50/37 -> 35/30
  for consistency. These are kinematic (viser viz; IK uses the .xml), so no mass/battery added;
  d435 was already present.

File: src/holosoma/holosoma/data/robots/g1/main_mesh_collision_halfspherehand.urdf (robot description, URDF)
Before this commit: robot g1, 42 links, 41 joints
Links:
- added link battery, mass 2.5
- added link d435_link
Joints:
- added joint battery_joint: type fixed, parent imu_in_torso, child battery, origin xyz=0.05 0.025 -0.01 rpy=0 0 0
- added joint d435_joint: type fixed, parent torso_link, child d435_link, origin xyz=0.0576235 0.01753 0.42987 rpy=0 0.8307767239493009 0
- joint left_ankle_pitch_joint: limit lower=-0.87267 upper=0.5236 effort=50 velocity=37 -> lower=-0.87267 upper=0.5236 effort=35 velocity=30
- joint left_ankle_roll_joint: limit lower=-0.2618 upper=0.2618 effort=50 velocity=37 -> lower=-0.2618 upper=0.2618 effort=35 velocity=30
- joint right_ankle_pitch_joint: limit lower=-0.87267 upper=0.5236 effort=50 velocity=37 -> lower=-0.87267 upper=0.5236 effort=35 velocity=30
- joint right_ankle_roll_joint: limit lower=-0.2618 upper=0.2618 effort=50 velocity=37 -> lower=-0.2618 upper=0.2618 effort=35 velocity=30

File: src/holosoma_retargeting/holosoma_retargeting/models/g1/g1_27dof.urdf (robot description, URDF)
Before this commit: robot g1_29dof, 55 links, 54 joints
Joints:
- joint left_ankle_pitch_joint: limit lower=-0.87267 upper=0.5236 effort=50 velocity=37 -> lower=-0.87267 upper=0.5236 effort=35 velocity=30
- joint left_ankle_roll_joint: limit lower=-0.2618 upper=0.2618 effort=50 velocity=37 -> lower=-0.2618 upper=0.2618 effort=35 velocity=30
- joint right_ankle_pitch_joint: limit lower=-0.87267 upper=0.5236 effort=50 velocity=37 -> lower=-0.87267 upper=0.5236 effort=35 velocity=30
- joint right_ankle_roll_joint: limit lower=-0.2618 upper=0.2618 effort=50 velocity=37 -> lower=-0.2618 upper=0.2618 effort=35 velocity=30

File: src/holosoma_retargeting/holosoma_retargeting/models/g1/g1_29dof.urdf (robot description, URDF)
Before this commit: robot g1_29dof, 55 links, 54 joints
Joints:
- joint left_ankle_pitch_joint: limit lower=-0.87267 upper=0.5236 effort=50 velocity=37 -> lower=-0.87267 upper=0.5236 effort=35 velocity=30
- joint left_ankle_roll_joint: limit lower=-0.2618 upper=0.2618 effort=50 velocity=37 -> lower=-0.2618 upper=0.2618 effort=35 velocity=30
- joint right_ankle_pitch_joint: limit lower=-0.87267 upper=0.5236 effort=50 velocity=37 -> lower=-0.87267 upper=0.5236 effort=35 velocity=30
- joint right_ankle_roll_joint: limit lower=-0.2618 upper=0.2618 effort=50 velocity=37 -> lower=-0.2618 upper=0.2618 effort=35 velocity=30

File: src/holosoma_retargeting/holosoma_retargeting/models/g1/g1_29dof_spherehand.urdf (robot description, URDF)
Before this commit: robot g1_29dof, 53 links, 52 joints
Joints:
- joint left_ankle_pitch_joint: limit lower=-0.87267 upper=0.5236 effort=50 velocity=37 -> lower=-0.87267 upper=0.5236 effort=35 velocity=30
- joint left_ankle_roll_joint: limit lower=-0.2618 upper=0.2618 effort=50 velocity=37 -> lower=-0.2618 upper=0.2618 effort=35 velocity=30
- joint right_ankle_pitch_joint: limit lower=-0.87267 upper=0.5236 effort=50 velocity=37 -> lower=-0.87267 upper=0.5236 effort=35 velocity=30
- joint right_ankle_roll_joint: limit lower=-0.2618 upper=0.2618 effort=50 velocity=37 -> lower=-0.2618 upper=0.2618 effort=35 velocity=30
